Commit message: Repository updated

File: urdf/robot2_laser.xacro (robot description, xacro)
@@ -1,5 +1,5 @@
 <?xml version="1.0"?>
-<robot xmlns:xacro="http://www.ros.org/wiki/xacro" name="robot2_xacro">
-<xacro:include filename="$(find robot1_description)/urdf/robot2.gazebo"/>
+<robot xmlns:xacro="http://www.ros.org/wiki/xacro" name="robot2_laser_xacro">
+<xacro:include filename="$(find robot1_description)/urdf/robot2_laser.gazebo"/>
 	<xacro:property name="length_wheel" value="0.04" />
 	<xacro:property name="radius_wheel" value="0.1" />
@@ -62,24 +62,12 @@
     </visual>
     <!-- caster front -->
-    <collision name="caster_front_collision">
-      <origin rpy=" 0 0 0" xyz="0.35 0 -0.05"/>
-      <geometry>
-        <sphere radius="0.05"/>
-      </geometry>
-    </collision>
-    <visual name="caster_front_visual">
-      <origin rpy=" 0 0 0" xyz="0.2 0 -0.05"/>
-      <geometry>
-        <sphere radius="0.05"/>
-      </geometry>
-    </visual>
   </link>
-   <link name="link_right_wheel">
+   <link name="link_back_right_wheel">
     <xacro:default_inertial mass="0.2"/>
-    <collision name="link_right_wheel_collision">
+    <collision name="link_back_right_wheel_collision">
       <origin rpy="0 1.5707 1.5707" xyz="0 0 0"/>
       <xacro:wheel_geometry />
     </collision>
-    <visual name="link_right_wheel_visual">
+    <visual name="link_back_right_wheel_visual">
       <origin rpy="0 1.5707 1.5707" xyz="0 0 0"/>
       <xacro:wheel_geometry />
@@ -87,11 +75,11 @@
     </visual>
   </link>
-   <link name="link_left_wheel">
+   <link name="link_back_left_wheel">
     <xacro:default_inertial mass="0.2"/>
-    <collision name="link_left_wheel_collision">
+    <collision name="link_back_left_wheel_collision">
       <origin rpy="0 1.5707 1.5707" xyz="0 0 0"/>
       <xacro:wheel_geometry />
     </collision>
-    <visual name="link_left_wheel_visual">
+    <visual name="link_back_left_wheel_visual">
       <origin rpy="0 1.5707 1.5707" xyz="0 0 0"/>
       <xacro:wheel_geometry />
@@ -99,7 +87,31 @@
     </visual>
   </link>
-  <joint name="joint_right_wheel" type="continuous">
-    <origin rpy="0 0 0" xyz="-0.05 0.15 0"/>
-    <child link="link_right_wheel"/>
+   <link name="link_front_right_wheel">
+    <xacro:default_inertial mass="0.2"/>
+    <collision name="link_front_right_wheel_collision">
+      <origin rpy="0 1.5707 1.5707" xyz="0 0 0"/>
+      <xacro:wheel_geometry />
+    </collision>
+    <visual name="link_front_right_wheel_visual">
+      <origin rpy="0 1.5707 1.5707" xyz="0 0 0"/>
+      <xacro:wheel_geometry />
+      <material name="red"/>
+    </visual>
+  </link>
+   <link name="link_front_left_wheel">
+    <xacro:default_inertial mass="0.2"/>
+    <collision name="link_front_left_wheel_collision">
+      <origin rpy="0 1.5707 1.5707" xyz="0 0 0"/>
+      <xacro:wheel_geometry />
+    </collision>
+    <visual name="link_front_left_wheel_visual">
+      <origin rpy="0 1.5707 1.5707" xyz="0 0 0"/>
+      <xacro:wheel_geometry />
+      <material name="red"/>
+    </visual>
+  </link>
+  <joint name="joint_back_right_wheel" type="continuous">
+    <origin rpy="0 0 0" xyz="-0.20 0.15 0"/>
+    <child link="link_back_right_wheel"/>
     <parent link="link_chassis"/>
     <axis rpy="0 0 0" xyz="0 1 0"/>
@@ -107,7 +119,7 @@
     <joint_properties damping="1.0" friction="1.0"/>
   </joint>
-  <joint name="joint_left_wheel" type="continuous">
-    <origin rpy="0 0 0" xyz="-0.05 -0.15 0"/>
-    <child link="link_left_wheel"/>
+  <joint name="joint_back_left_wheel" type="continuous">
+    <origin rpy="0 0 0" xyz="-0.20 -0.15 0"/>
+    <child link="link_back_left_wheel"/>
     <parent link="link_chassis"/>
     <axis rpy="0 0 0" xyz="0 1 0"/>
@@ -115,5 +127,21 @@
     <joint_properties damping="1.0" friction="1.0"/>
   </joint>
-  <link name="camera_link">
+  <joint name="joint_front_right_wheel" type="continuous">
+    <origin rpy="0 0 0" xyz="0.20 0.15 0"/>
+    <child link="link_front_right_wheel"/>
+    <parent link="link_chassis"/>
+    <axis rpy="0 0 0" xyz="0 1 0"/>
+    <limit effort="10000" velocity="1000"/>
+    <joint_properties damping="1.0" friction="1.0"/>
+  </joint>
+  <joint name="joint_front_left_wheel" type="continuous">
+    <origin rpy="0 0 0" xyz="0.20 -0.15 0"/>
+    <child link="link_front_left_wheel"/>
+    <parent link="link_chassis"/>
+    <axis rpy="0 0 0" xyz="0 1 0"/>
+    <limit effort="10000" velocity="1000"/>
+    <joint_properties damping="1.0" friction="1.0"/>
+  </joint>
+   <link name="hokuyo_link">
 	    <collision>
 	      <origin xyz="0 0 0.025" rpy="0 0 0"/>
@@ -136,10 +164,10 @@
 	      <inertia ixx="1e-6" ixy="0" ixz="0" iyy="1e-6" iyz="0" izz="1e-6" />
 	    </inertial>
-  </link>
-  <joint name="camera_joint" type="fixed">
+ 	 </link>
+ 	 <joint name="hokuyo_joint" type="fixed">
 	    <axis xyz="0 1 0" />
-	    <origin xyz="0.23 0 0.0" rpy="0 0 0"/>
+	    <origin xyz="0.28 0 0.05" rpy="0 0 0"/>
 	    <parent link="link_chassis"/>
-	    <child link="camera_link"/>
+	    <child link="hokuyo_link"/>
 	 </joint>
 </robot>
